File: modules/PGTN014_percussive_synthesiser/PGTN014_percussive_synth.sch (EAGLE design)
At the start: 207 parts, among them IC1 LM13700N, IC2 LM13700N, IC3 LM13700N, IC4 4046N, IC5 XR-2206, IC6 TL074P, Q1 2N3904, Q10 2N3906, Q11 2N3906, Q12 2N3906, Q13 2N3906, Q14 2N3906, Q2 2N3904, Q3 2N3904, Q4 2N3904, Q5 2N3904, Q6 2N3904, Q7 2N3904, Q8 2N3906, Q9 2N3904

Commit message: added sequencer
Parts:
- Q9: value 2N3904 -> 2N3906; device transistors:2N3904 -> transistors:2N3906
- R16: value 10k -> 1k
- R35: value 20k -> 10k
- R36: value (none) -> 10k
Connections:
- removed net PE: IC6D.+IN, R35.2
- net GND: now also IC6D.+IN, R35.2

Commit message: Fix for following issues * Pin 12 of IC5 shorted to pin 10. Pin 12 should be GND, but not pin 10 so have to kludge on IC pin. * SHL_SWP3 should connect to GND. No big deal as can just connect pot directly to GND instead. * Pin 12 of IC6 not connected to GND. * Pin 3 and 4 of IC1 swapped.
Connections:
- removed net N$105: C31.+, IC5.10, IC5.12
- removed net N$70: R39.E, SHL_SWP3.3
- new net N$113: C31.-, IC5.10
- net GND: now also C31.+, IC5.12, R39.E, SHL_SWP3.3; no longer C31.-
- net N$25: now also IC1OTA1.IN_P; no longer IC1OTA1.IN_N
- net N$30: now also IC1OTA1.IN_N; no longer IC1OTA1.IN_P
Other:
- moved on the sheet: C31, IC1OTA1
Changed lines of the file:
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@@
 </part>
 <part name="Q9" library="transistors" deviceset="2N3906" device=""/>
+<part name="SUPPLY95" library="supply" deviceset="GND" device="">
+<attribute name="SPICEPREFIX" value="G"/>
+</part>
 </parts>
 <sheets>
@@
 <instance part="SUPPLY16" gate="+12V" x="137.16" y="76.2"/>
 <instance part="R47" gate="G$1" x="195.58" y="40.64" rot="R180"/>
-<instance part="IC1" gate="OTA1" x="162.56" y="134.62"/>
+<instance part="IC1" gate="OTA1" x="162.56" y="134.62" rot="MR180"/>
 <instance part="IC1" gate="BUF1" x="198.12" y="132.08"/>
 <instance part="IC1" gate="OTA2" x="243.84" y="134.62"/>
@@
 <instance part="SUPPLY89" gate="+12V" x="281.94" y="-350.52"/>
 <instance part="C15" gate="G$1" x="302.26" y="-365.76" rot="R270"/>
-<instance part="C31" gate="G$1" x="347.98" y="-386.08"/>
-<instance part="SUPPLY90" gate="GND" x="347.98" y="-393.7"/>
+<instance part="C31" gate="G$1" x="340.36" y="-370.84" rot="R270"/>
+<instance part="SUPPLY90" gate="GND" x="347.98" y="-396.24"/>
 <instance part="IMP_OUT" gate="HEADER" x="264.16" y="-167.64" rot="R180"/>
 <instance part="NSE_OUT" gate="HEADER" x="353.06" y="58.42" rot="R180"/>
@@
 <instance part="SUPPLY94" gate="G$1" x="266.7" y="58.42"/>
 <instance part="Q9" gate="G$1" x="294.64" y="45.72" rot="R180"/>
+<instance part="SUPPLY95" gate="GND" x="137.16" y="-342.9"/>
 </instances>
 <busses>
@@
 </segment>
 <segment>
-<pinref part="C31" gate="G$1" pin="-"/>
-<pinref part="SUPPLY90" gate="GND" pin="PE"/>
-</segment>
-<segment>
 <pinref part="IC6" gate="D" pin="+IN"/>
 <pinref part="SUPPLY91" gate="GND" pin="PE"/>
@@
 <pinref part="SUPPLY92" gate="GND" pin="PE"/>
 <wire x1="416.56" y1="-106.68" x2="416.56" y2="-104.14" width="0.1524" layer="91"/>
+</segment>
+<segment>
+<pinref part="R39" gate="G$1" pin="E"/>
+<pinref part="SHL_SWP3" gate="HEADER" pin="3"/>
+<pinref part="SUPPLY95" gate="GND" pin="PE"/>
+<junction x="137.16" y="-340.36"/>
+<pinref part="SUPPLY95" gate="GND" pin="PE"/>
+<wire x1="137.16" y1="-340.36" x2="137.16" y2="-337.82" width="0.1524" layer="91"/>
+<junction x="137.16" y="-337.82"/>
+</segment>
+<segment>
+<pinref part="IC5" gate="G$1" pin="12"/>
+<wire x1="332.74" y1="-365.76" x2="347.98" y2="-365.76" width="0.1524" layer="91"/>
+<pinref part="SUPPLY90" gate="GND" pin="PE"/>
+<wire x1="347.98" y1="-393.7" x2="347.98" y2="-370.84" width="0.1524" layer="91"/>
+<pinref part="C31" gate="G$1" pin="+"/>
+<wire x1="347.98" y1="-370.84" x2="347.98" y2="-365.76" width="0.1524" layer="91"/>
+<wire x1="342.9" y1="-370.84" x2="347.98" y2="-370.84" width="0.1524" layer="91"/>
+<junction x="347.98" y="-370.84"/>
 </segment>
 </net>
@@
 <net name="N$18" class="0">
 <segment>
-<pinref part="IC1" gate="OTA1" pin="I_BIAS"/>
-<wire x1="170.18" y1="142.24" x2="177.8" y2="142.24" width="0.1524" layer="91"/>
-<wire x1="177.8" y1="142.24" x2="177.8" y2="93.98" width="0.1524" layer="91"/>
 <wire x1="177.8" y1="93.98" x2="193.04" y2="93.98" width="0.1524" layer="91"/>
 <pinref part="Q8" gate="G$1" pin="C"/>
@@
 <wire x1="259.08" y1="142.24" x2="251.46" y2="142.24" width="0.1524" layer="91"/>
 <junction x="193.04" y="93.98"/>
+<pinref part="IC1" gate="OTA1" pin="I_BIAS"/>
+<wire x1="170.18" y1="127" x2="170.18" y2="104.14" width="0.1524" layer="91"/>
+<wire x1="170.18" y1="104.14" x2="177.8" y2="104.14" width="0.1524" layer="91"/>
+<wire x1="177.8" y1="104.14" x2="177.8" y2="93.98" width="0.1524" layer="91"/>
 </segment>
 </net>
 <net name="N$19" class="0">
 <segment>
-<pinref part="IC1" gate="OTA1" pin="OUT"/>
 <pinref part="IC1" gate="BUF1" pin="B"/>
-<wire x1="175.26" y1="134.62" x2="187.96" y2="134.62" width="0.1524" layer="91"/>
 <pinref part="C1" gate="G$1" pin="2"/>
 <wire x1="187.96" y1="134.62" x2="190.5" y2="134.62" width="0.1524" layer="91"/>
 <wire x1="187.96" y1="127" x2="187.96" y2="134.62" width="0.1524" layer="91"/>
+<pinref part="IC1" gate="OTA1" pin="OUT"/>
+<wire x1="175.26" y1="134.62" x2="187.96" y2="134.62" width="0.1524" layer="91"/>
 <junction x="187.96" y="134.62"/>
 </segment>
@@
 <segment>
 <pinref part="R61" gate="G$1" pin="1"/>
-<pinref part="IC1" gate="OTA1" pin="IN_N"/>
 <wire x1="144.78" y1="132.08" x2="147.32" y2="132.08" width="0.1524" layer="91"/>
 <pinref part="R11" gate="G$1" pin="1"/>
+<wire x1="147.32" y1="129.54" x2="147.32" y2="132.08" width="0.1524" layer="91"/>
+<pinref part="IC1" gate="OTA1" pin="IN_P"/>
 <wire x1="147.32" y1="132.08" x2="154.94" y2="132.08" width="0.1524" layer="91"/>
-<wire x1="147.32" y1="129.54" x2="147.32" y2="132.08" width="0.1524" layer="91"/>
 <junction x="147.32" y="132.08"/>
 </segment>
@@
 <net name="N$30" class="0">
 <segment>
-<pinref part="IC1" gate="OTA1" pin="IN_P"/>
-<wire x1="154.94" y1="137.16" x2="152.4" y2="137.16" width="0.1524" layer="91"/>
 <wire x1="152.4" y1="137.16" x2="152.4" y2="154.94" width="0.1524" layer="91"/>
 <pinref part="R87" gate="G$1" pin="2"/>
@@
 <pinref part="R60" gate="G$1" pin="2"/>
 <wire x1="152.4" y1="154.94" x2="152.4" y2="157.48" width="0.1524" layer="91"/>
+<pinref part="IC1" gate="OTA1" pin="IN_N"/>
+<wire x1="154.94" y1="137.16" x2="152.4" y2="137.16" width="0.1524" layer="91"/>
 </segment>
 </net>
@@
 </segment>
 </net>
-<net name="N$70" class="0">
-<segment>
-<pinref part="R39" gate="G$1" pin="E"/>
-<pinref part="SHL_SWP3" gate="HEADER" pin="3"/>
-</segment>
-</net>
 <net name="N$71" class="0">
 <segment>
@@
 <pinref part="IC5" gate="G$1" pin="6"/>
 <wire x1="294.64" y1="-368.3" x2="317.5" y2="-368.3" width="0.1524" layer="91"/>
-</segment>
-</net>
-<net name="N$105" class="0">
-<segment>
-<pinref part="IC5" gate="G$1" pin="10"/>
-<wire x1="332.74" y1="-370.84" x2="347.98" y2="-370.84" width="0.1524" layer="91"/>
-<pinref part="C31" gate="G$1" pin="+"/>
-<wire x1="347.98" y1="-370.84" x2="347.98" y2="-383.54" width="0.1524" layer="91"/>
-<pinref part="IC5" gate="G$1" pin="12"/>
-<wire x1="332.74" y1="-365.76" x2="347.98" y2="-365.76" width="0.1524" layer="91"/>
-<wire x1="347.98" y1="-365.76" x2="347.98" y2="-370.84" width="0.1524" layer="91"/>
-<junction x="347.98" y="-370.84"/>
 </segment>
 </net>
@@
 </segment>
 </net>
+<net name="N$113" class="0">
+<segment>
+<pinref part="IC5" gate="G$1" pin="10"/>
+<pinref part="C31" gate="G$1" pin="-"/>
+<wire x1="335.28" y1="-370.84" x2="332.74" y2="-370.84" width="0.1524" layer="91"/>
+</segment>
+</net>
