File: modules/PGTN005_filter/PGTN005_filter.brd (EAGLE design)
At the start: 79.7 x 73.7 mm, 113 parts, among them IC1 TL084P, IC2 LM13700N, IC3 TL084P, IC4 TL082P, IC5 LM13700N, Q1 2N3904, Q2 2N3904, Q3 2N3906, Q4 2N3906

Commit message: Changed 1M input resistors to 300k in filter to increase gain.
Parts:
- R30, R31, R32: value 1M -> 300k
