File: blocks/PGTNX03_vcf/PGTNX03_vcf_bp_lp.sch (EAGLE design)
At the start: 70 parts, among them IC1 AS3320, IC2 TL084P

Commit message: Changes
Parts:
- added R29, R30, R31: 100k, controls_off_brd:POTENTIOMETER
Connections:
- new net PE: R29.E, R31.E
- net +12V: now also R29.A, R31.A
- net N$27: now also R31.S
- net N$30: now also R30.E
- net N$31: now also R29.S
- net N$4: now also R30.A
Other:
- note added: "RESONANCE CV"
