File: blocks/PGTNX05_daisy/PGTNX05_daisy2_main.sch (EAGLE design)
At the start: 164 parts, among them IC1 TL074P, IC2 7805TV, IC3 TL074P, IC4 MCP6004, IC5 MCP6004, IC6 TL074P, Q1 2N3904, Q2 2N3904, U1 DAISY, U2 LM4040-10V

Commit message: Changes
Parts:
- removed 27, 28, AIN1, AIN2, AOUT1, AOUT2, CVOUT1, CVOUT2: HEADER/MALE/01, connectors:HEADER/MALE/01
- removed C19, C27, C28: 100nF, capacitors:CAPACITORCERAMICDISC/5
- removed IC6: TL074P, ic_analogue:TL074P
- removed U2: LM4040-10V, ic_voltage_reg:LM4040CYM3-2.5
- added AINL1, AINL2, AINR1, AINR2, AOUTL1, AOUTR1, CV10A, CV10B, CV11A, CV11B, CV12A, CV12B, CV9A, CV9B: HEADER/MALE/01, connectors:HEADER/MALE/01
- added C29: 0.1uF, capacitors:CAPACITOR/POLARIZEDE2.5-6
- added IC7: 79L05, linear:79L05Z
- added IC8: LM4040-5V, ic_voltage_reg:LM4040
- C1, C2: value 10uF -> 0.33uF
- C10, C11, C7: value 47pF -> 1nF
- C14: value 100nF -> 1nF
- C6: value 47pF -> 100nF
- IC3: value TL074P -> MCP6004
- R15, R64, R8: value 100k -> 33k
- R29: value 2k -> 100k
- R65, R67: value 49.9k -> 100k
- R69: value 33k -> 100k
- R7: value 100k -> 2K
- R70, R71: value 1k -> 100k
Connections:
- removed net 25_GTIN1: R54.2, U1.GPIO26(SAI2_SD_B)
- removed net 27: 27.3, U1.GPIO28(SAI2_FS_B)
- removed net 28: 28.3, U1.GPIO29(SAI2_SCK_B)
- removed net DAC1: R68.1, U1.GPIO24(DAC1_OUT1)
- removed net DAC2: R69.1, U1.GPIO23(DAC1_OUT2)
- removed net N$72: IC6C.-IN, R62.2, R66.1
- removed net N$73: IC6D.-IN, R67.1, R69.2
- removed net N$74: IC6C.OUT, R66.2, R71.1
- removed net N$75: IC6B.OUT, R64.2, R70.1
- removed net N$76: IC6A.-IN, R65.1, R68.2
- removed net N$77: CVOUT1.3, R70.2
- removed net N$78: CVOUT2.3, R71.2
- new net 27_GTIN1: R54.2, U1.GPIO28(SAI2_FS_B)
- new net ADC10: C11.2, IC3C.OUT, R64.2, U1.GPIO26(SAI2_SD_B)
- new net ADC11: C14.2, IC3D.OUT, R68.2, U1.GPIO29(SAI2_SCK_B)
- new net ADC7: C25.2, IC5D.OUT, R50.2, U1.GPIO23(DAC1_OUT2)
- new net ADC8: C7.2, IC3A.OUT, R8.2, U1.GPIO24(DAC1_OUT1)
- new net N$57: C14.1, IC3D.-IN, R68.1, R69.2, R70.2, R71.2
- new net N$60: CV12A.3, R69.1
- new net N$68: CV12B.3, R70.1
- net +12V: no longer C15.2, C27.2, IC3P.V+, IC6P.V+
- net -12V: now also IC7.VI, R7.2; no longer C14.1, C28.1, IC3P.V-, IC6P.V-, R29.2
- net -5VREF: now also C29.-, C6.2, IC7.VO, IC8.A, R13.1, R67.1, R7.1, R71.1; no longer C19.2, U2.A
- net 3.3VA: now also C15.2, IC3P.V+
- net ADC9: now also C10.2, IC3B.OUT, R15.2; no longer C25.2, IC5D.OUT, R50.2
- net N$10: now also IC1A.OUT; no longer IC1B.OUT
- net N$11: now also AOUTR1.3; no longer AOUT1.3
- net N$12: now also IC1C.OUT, R19.1; no longer IC3B.OUT, R12.1
- net N$13: now also CV9B.3, R12.1; no longer C6.1, IC1A.-IN, R4.1, R7.2
- net N$14: now also CV9A.3, R11.1; no longer C10.1, IC3A.-IN, R12.2, R13.1
- net N$15: now also IC1D.OUT, R20.1; no longer IC3C.OUT, R11.1
- net N$16: now also C10.1, IC3B.-IN, R29.2, R62.2, R63.2; no longer C11.1, IC3D.-IN, R11.2
- net N$17: now also IC1D.-IN; no longer IC3C.-IN
- net N$18: now also CV10A.3, R62.1; no longer C11.2, IC3D.OUT, R15.2, R20.1
- net N$19: now also CV10B.3, R63.1; no longer C10.2, IC3A.OUT, R13.2, R19.1
- net N$2: now also AINR2.3, R4.1; no longer C7.2, IC1D.OUT, R1.1, R6.2
- net N$20: now also IC1C.-IN; no longer IC3B.-IN
- net N$21: now also AOUTL1.3; no longer AOUT2.3
- net N$3: now also AINL2.3, R6.1; no longer C6.2, IC1A.OUT, R2.1, R4.2
- net N$4: now also IC1A.-IN, R4.2; no longer IC1B.-IN
- net N$5: now also IC1B.-IN, R6.2; no longer IC1C.-IN
- net N$6: now also AINR1.3, R2.1; no longer AIN1.3, R7.1
- net N$69: now also CV11B.3, R66.1; no longer IC6A.OUT, R63.1, R65.2
- net N$7: now also AINL1.3, R1.1; no longer AIN2.3, R8.1
- net N$70: now also CV11A.3, R65.1; no longer IC6B.-IN, R63.2, R64.1
- net N$71: now also C11.1, IC3C.-IN, R64.1, R65.2, R66.2; no longer IC6D.OUT, R62.1
- net N$8: now also IC3A.-IN, R11.2, R12.2, R13.2, R8.1; no longer IC1D.-IN, R6.1, R8.2
- net N$9: now also IC1B.OUT; no longer IC1C.OUT
- net PE: now also C29.+, C6.1, IC3P.V-, IC7.GND, IC8.C; no longer C14.2, C19.1, C27.1, C28.2, IC6A.+IN, IC6B.+IN, IC6C.+IN, IC6D.+IN, U2.C
Other:
- moved on the sheet: -5V, C10, C11, C14, C15, C6, C7, GTIN1, GTIN2, IC1A, IC1B, IC1C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
