File: breakout/jack10_breakout.brd (EAGLE design)
At the start: 13 x 14.1 mm, 5 parts

Commit message: Changes
Parts:
- added NORM1, NORM2, NORM3, NORM4, NORM5, NORM6, NORM7, NORM8, NORM9, SIG1, SIG2, SIG3, SIG4, SIG5, SIG6, SIG7, SIG8, SIG9: HEADER/MALE/01, connectors:HEADER/MALE/01
- added U$10, U$2, U$3, U$4, U$5, U$6, U$7, U$8, U$9: WQP-PJ301M-12_JACK, controls:WQP-PJ301M-12_JACK
- moved GND1 14.2 mm to (3.81, 21.6), turned to 90 degrees
Connections:
- removed net N$6: GND.1, GND1.1, U$1.P$3
- new net N$10: SIG3.1, U$4.P$1
- new net N$11: NORM3.1, U$4.P$2
- new net N$12: GND.1, GND1.1, U$1.P$3, U$10.P$3, U$2.P$3, U$3.P$3, U$4.P$3, U$5.P$3, U$6.P$3, U$7.P$3, U$8.P$3, U$9.P$3
- new net N$13: SIG4.1, U$5.P$1
- new net N$14: NORM4.1, U$5.P$2
- new net N$16: SIG5.1, U$6.P$1
- new net N$17: NORM5.1, U$6.P$2
- new net N$19: SIG6.1, U$7.P$1
- new net N$20: NORM6.1, U$7.P$2
- new net N$22: SIG7.1, U$8.P$1
- new net N$23: NORM7.1, U$8.P$2
- new net N$25: SIG8.1, U$9.P$1
- new net N$26: NORM8.1, U$9.P$2
- new net N$28: SIG9.1, U$10.P$1
- new net N$29: NORM9.1, U$10.P$2
- new net N$4: SIG1.1, U$2.P$1
- new net N$5: NORM1.1, U$2.P$2
- new net N$7: SIG2.1, U$3.P$1
- new net N$8: NORM2.1, U$3.P$2
Routing:
- net N$12: track 0.00 -> 123.8 mm
- net N$7: track 0.00 -> 13.5 mm
- net N$4: track 0.00 -> 13.5 mm
- net N$28: track 0.00 -> 13.5 mm
- net N$25: track 0.00 -> 13.5 mm
- net N$22: track 0.00 -> 13.5 mm
- net N$19: track 0.00 -> 13.5 mm
- net N$16: track 0.00 -> 13.5 mm
- net N$13: track 0.00 -> 13.5 mm
- net N$10: track 0.00 -> 13.5 mm
- net N$6: track 5.14 -> 0.00 mm
- net N$29: track 0.00 -> 3.90 mm
- net N$26: track 0.00 -> 3.90 mm
- net N$23: track 0.00 -> 3.90 mm
- net N$20: track 0.00 -> 3.90 mm
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Other:
- board size 13 x 14.1 mm -> 58.7 x 28.1 mm
