File: breakout/jack10_breakout.sch (EAGLE design)
At the start: 5 parts

Commit message: Changes
Parts:
- added NORM1, NORM2, NORM3, NORM4, NORM5, NORM6, NORM7, NORM8, NORM9, SIG1, SIG2, SIG3, SIG4, SIG5, SIG6, SIG7, SIG8, SIG9: HEADER/MALE/01, connectors:HEADER/MALE/01
- added U$10, U$2, U$3, U$4, U$5, U$6, U$7, U$8, U$9: WQP-PJ301M-12_JACK, controls:WQP-PJ301M-12_JACK
Connections:
- removed net N$6: GND.3, GND1.3, U$1.1
- new net N$10: SIG3.3, U$4.2
- new net N$11: NORM3.3, U$4.3
- new net N$12: GND.3, GND1.3, U$1.1, U$10.1, U$2.1, U$3.1, U$4.1, U$5.1, U$6.1, U$7.1, U$8.1, U$9.1
- new net N$13: SIG4.3, U$5.2
- new net N$14: NORM4.3, U$5.3
- new net N$16: SIG5.3, U$6.2
- new net N$17: NORM5.3, U$6.3
- new net N$19: SIG6.3, U$7.2
- new net N$20: NORM6.3, U$7.3
- new net N$22: SIG7.3, U$8.2
- new net N$23: NORM7.3, U$8.3
- new net N$25: SIG8.3, U$9.2
- new net N$26: NORM8.3, U$9.3
- new net N$28: SIG9.3, U$10.2
- new net N$29: NORM9.3, U$10.3
- new net N$4: SIG1.3, U$2.2
- new net N$5: NORM1.3, U$2.3
- new net N$7: SIG2.3, U$3.2
- new net N$8: NORM2.3, U$3.3
