File: breakout/potentiometer_breakout.sch (EAGLE design)
At the start: 5 parts

Commit message: Changes
Parts:
- removed GND, GND1, NORM, SIG: HEADER/MALE/01, connectors:HEADER/MALE/01
- removed U$1: WQP-PJ301M-12_JACK, controls:WQP-PJ301M-12_JACK
- added 1, 2, 3: HEADER/MALE/01, connectors:HEADER/MALE/01
- added VR1: (no value), controls:9MM_SNAP-IN_POT_
Connections:
- removed net N$6: GND.3, GND1.3, U$1.1
- new net N$3: 3.3, VR1.A
- net N$1: now also 1.3, VR1.E; no longer SIG.3, U$1.2
- net N$2: now also 2.3, VR1.S; no longer NORM.3, U$1.3
Changed lines of the file:
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@@
 </classes>
 <parts>
-<part name="GND" library="connectors" deviceset="HEADER/MALE/01" device=""/>
-<part name="NORM" library="connectors" deviceset="HEADER/MALE/01" device=""/>
-<part name="SIG" library="connectors" deviceset="HEADER/MALE/01" device=""/>
-<part name="U$1" library="controls" deviceset="WQP-PJ301M-12_JACK" device=""/>
-<part name="GND1" library="connectors" deviceset="HEADER/MALE/01" device=""/>
+<part name="2" library="connectors" deviceset="HEADER/MALE/01" device=""/>
+<part name="VR1" library="controls" deviceset="9MM_SNAP-IN_POT" device="_"/>
+<part name="1" library="connectors" deviceset="HEADER/MALE/01" device=""/>
+<part name="3" library="connectors" deviceset="HEADER/MALE/01" device=""/>
 </parts>
 <sheets>
@@
 </plain>
 <instances>
-<instance part="GND" gate="HEADER" x="7.62" y="111.76" smashed="yes">
-<attribute name="NAME" x="-6.096" y="110.744" size="1.778" layer="96"/>
+<instance part="2" gate="HEADER" x="66.04" y="86.36" smashed="yes" rot="R180">
+<attribute name="NAME" x="79.756" y="87.376" size="1.778" layer="96" rot="R180"/>
 </instance>
-<instance part="NORM" gate="HEADER" x="7.62" y="114.3" smashed="yes">
-<attribute name="NAME" x="-6.096" y="113.284" size="1.778" layer="96"/>
+<instance part="VR1" gate="G$1" x="58.42" y="86.36" smashed="yes">
+<attribute name="NAME" x="53.34" y="83.82" size="1.778" layer="95" rot="R90"/>
+<attribute name="VALUE" x="55.88" y="83.82" size="1.778" layer="96" rot="R90"/>
 </instance>
-<instance part="SIG" gate="HEADER" x="7.62" y="116.84" smashed="yes">
-<attribute name="NAME" x="-6.096" y="115.824" size="1.778" layer="96"/>
+<instance part="1" gate="HEADER" x="60.96" y="93.98" smashed="yes" rot="R180">
+<attribute name="NAME" x="74.676" y="94.996" size="1.778" layer="96" rot="R180"/>
 </instance>
-<instance part="U$1" gate="G$1" x="20.32" y="114.3" smashed="yes">
-<attribute name="NAME" x="17.78" y="118.364" size="1.778" layer="95"/>
-<attribute name="VALUE" x="17.78" y="108.204" size="1.778" layer="96"/>
-</instance>
-<instance part="GND1" gate="HEADER" x="7.62" y="109.22" smashed="yes">
-<attribute name="NAME" x="-6.096" y="108.204" size="1.778" layer="96"/>
+<instance part="3" gate="HEADER" x="60.96" y="78.74" smashed="yes" rot="R180">
+<attribute name="NAME" x="74.676" y="79.756" size="1.778" layer="96" rot="R180"/>
 </instance>
 </instances>
@@
 <net name="N$1" class="0">
 <segment>
-<pinref part="U$1" gate="G$1" pin="2"/>
-<pinref part="SIG" gate="HEADER" pin="3"/>
-<wire x1="10.16" y1="116.84" x2="15.24" y2="116.84" width="0.1524" layer="91"/>
+<pinref part="VR1" gate="G$1" pin="E"/>
+<pinref part="1" gate="HEADER" pin="3"/>
 </segment>
 </net>
 <net name="N$2" class="0">
 <segment>
-<pinref part="U$1" gate="G$1" pin="3"/>
-<pinref part="NORM" gate="HEADER" pin="3"/>
-<wire x1="10.16" y1="114.3" x2="15.24" y2="114.3" width="0.1524" layer="91"/>
+<pinref part="VR1" gate="G$1" pin="S"/>
+<pinref part="2" gate="HEADER" pin="3"/>
 </segment>
 </net>
-<net name="N$6" class="0">
+<net name="N$3" class="0">
 <segment>
-<pinref part="U$1" gate="G$1" pin="1"/>
-<pinref part="GND" gate="HEADER" pin="3"/>
-<wire x1="10.16" y1="111.76" x2="12.7" y2="111.76" width="0.1524" layer="91"/>
-<pinref part="GND1" gate="HEADER" pin="3"/>
-<wire x1="12.7" y1="111.76" x2="15.24" y2="111.76" width="0.1524" layer="91"/>
-<wire x1="10.16" y1="109.22" x2="12.7" y2="109.22" width="0.1524" layer="91"/>
-<wire x1="12.7" y1="109.22" x2="12.7" y2="111.76" width="0.1524" layer="91"/>
-<junction x="12.7" y="111.76"/>
+<pinref part="VR1" gate="G$1" pin="A"/>
+<pinref part="3" gate="HEADER" pin="3"/>
 </segment>
 </net>
